File: 1. Power Submodule/Group22_Power/Sensors.kicad_sch (KiCad schematic)
At the start: 0 parts

Commit message: power pcb
Parts:
- added J?: Conn_01x02_Male, Connector_PinHeader_2.54mm:PinHeader_1x02_P2.54mm_Vertical, symbol Connector:Conn_01x02_Male
- added R? (x2): 10k, Resistor_SMD:R_0402_1005Metric, symbol Device:R
- added U?: SHT30-DIS, Sensor_Humidity:Sensirion_DFN-8-1EP_2.5x2.5mm_P0.5mm_EP1.1x1.7mm, symbol Sensor_Humidity:SHT30-DIS
Connections:
- new net +3V3REG: R?.1, R?.1, U?.5 (VDD)
- new net GND: U?.2 (ADDR), U?.7 (R), U?.8 (VSS), U?.9 (VSS)
- new net SCL: J?.1 (Pin_1), R?.2, U?.4 (SCL)
- new net SDA: J?.2 (Pin_2), R?.2, U?.1 (SDA)
- no-connect marks 0 -> 2
Other:
- note added: "On-board Temperature and Humidity Sensor"
Changed lines of the file:
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@@
 (kicad_sch (version 20211123) (generator eeschema)
   (paper "A4")
+  (junction (at 208.915 143.51) (diameter 0) (color 0 0 0 0)
+  )
+  (junction (at 217.805 146.05) (diameter 0) (color 0 0 0 0)
+  )
+  (junction (at 208.915 125.73) (diameter 0) (color 0 0 0 0)
+  )
+  (junction (at 193.675 125.73) (diameter 0) (color 0 0 0 0)
+  )
+  (junction (at 180.34 148.59) (diameter 0) (color 0 0 0 0)
+  )
+  (no_connect (at 183.515 146.05))
+  (no_connect (at 203.835 148.59))
+  (wire (pts (xy 180.34 143.51) (xy 183.515 143.51))
+    (stroke (width 0) (type default) (color 0 0 0 0))
+  )
+  (wire (pts (xy 193.675 125.73) (xy 208.915 125.73))
+    (stroke (width 0) (type default) (color 0 0 0 0))
+  )
+  (wire (pts (xy 180.34 153.67) (xy 180.34 148.59))
+    (stroke (width 0) (type default) (color 0 0 0 0))
+  )
+  (wire (pts (xy 208.915 125.73) (xy 208.915 131.445))
+    (stroke (width 0) (type default) (color 0 0 0 0))
+  )
+  (wire (pts (xy 208.915 143.51) (xy 226.695 143.51))
+    (stroke (width 0) (type default) (color 0 0 0 0))
+  )
+  (wire (pts (xy 180.34 148.59) (xy 180.34 143.51))
+    (stroke (width 0) (type default) (color 0 0 0 0))
+  )
+  (wire (pts (xy 217.805 146.05) (xy 203.835 146.05))
+    (stroke (width 0) (type default) (color 0 0 0 0))
+  )
+  (wire (pts (xy 180.34 148.59) (xy 183.515 148.59))
+    (stroke (width 0) (type default) (color 0 0 0 0))
+  )
+  (wire (pts (xy 217.805 125.73) (xy 208.915 125.73))
+    (stroke (width 0) (type default) (color 0 0 0 0))
+  )
+  (wire (pts (xy 203.835 143.51) (xy 208.915 143.51))
+    (stroke (width 0) (type default) (color 0 0 0 0))
+  )
+  (wire (pts (xy 217.805 131.445) (xy 217.805 125.73))
+    (stroke (width 0) (type default) (color 0 0 0 0))
+  )
+  (wire (pts (xy 193.675 138.43) (xy 193.675 125.73))
+    (stroke (width 0) (type default) (color 0 0 0 0))
+  )
+  (wire (pts (xy 208.915 139.065) (xy 208.915 143.51))
+    (stroke (width 0) (type default) (color 0 0 0 0))
+  )
+  (wire (pts (xy 217.805 139.065) (xy 217.805 146.05))
+    (stroke (width 0) (type default) (color 0 0 0 0))
+  )
+  (wire (pts (xy 217.805 146.05) (xy 226.695 146.05))
+    (stroke (width 0) (type default) (color 0 0 0 0))
+  )
+  (wire (pts (xy 193.675 125.73) (xy 185.42 125.73))
+    (stroke (width 0) (type default) (color 0 0 0 0))
+  )
+  (text "On-board Temperature and Humidity Sensor" (at 173.99 123.19 0)
+    (effects (font (size 2 2) (thickness 0.4) bold) (justify left bottom))
+  )
+  (label "SCL" (at 222.885 146.05 0)
+    (effects (font (size 1.27 1.27)) (justify left bottom))
+  )
+  (label "SDA" (at 222.885 143.51 0)
+    (effects (font (size 1.27 1.27)) (justify left bottom))
+  )
+  (global_label "+3V3REG" (shape input) (at 185.42 125.73 180) (fields_autoplaced)
+    (effects (font (size 1.27 1.27)) (justify right))
+    (property "Intersheet References" "${INTERSHEET_REFS}" (id 0) (at 174.3268 125.8094 0)
+      (effects (font (size 1.27 1.27)) (justify right) hide)
+    )
+  )
+  (symbol (lib_id "power:GND") (at 193.675 153.67 0) (unit 1)
+    (in_bom yes) (on_board yes) (fields_autoplaced)
+    (property "Reference" "#PWR?" (id 0) (at 193.675 160.02 0)
+      (effects (font (size 1.27 1.27)) hide)
+    )
+    (property "Value" "GND" (id 1) (at 193.675 158.115 0))
+    (property "Footprint" "" (id 2) (at 193.675 153.67 0)
+      (effects (font (size 1.27 1.27)) hide)
+    )
+    (property "Datasheet" "" (id 3) (at 193.675 153.67 0)
+      (effects (font (size 1.27 1.27)) hide)
+    )
+    (pin "1")
+  )
+  (symbol (lib_id "Sensor_Humidity:SHT30-DIS") (at 193.675 146.05 0) (unit 1)
+    (in_bom yes) (on_board yes) (fields_autoplaced)
+    (property "Reference" "U?" (id 0) (at 195.6944 135.89 0)
+      (effects (font (size 1.27 1.27)) (justify left))
+    )
+    (property "Value" "SHT30-DIS" (id 1) (at 195.6944 138.43 0)
+      (effects (font (size 1.27 1.27)) (justify left))
+    )
+    (property "Footprint" "Sensor_Humidity:Sensirion_DFN-8-1EP_2.5x2.5mm_P0.5mm_EP1.1x1.7mm" (id 2) (at 193.675 144.78 0)
+      (effects (font (size 1.27 1.27)) hide)
+    )
+    (property "Datasheet" "https://datasheet.lcsc.com/lcsc/2106070104_Sensirion-SHT30-DIS-B10KS_C2687423.pdf" (id 3) (at 193.675 144.78 0)
+      (effects (font (size 1.27 1.27)) hide)
+    )
+    (property "Alt_LCSC" "C77361" (id 4) (at 193.675 146.05 0)
+      (effects (font (size 1.27 1.27)) hide)
+    )
+    (property "Extended" "1" (id 5) (at 193.675 146.05 0)
+      (effects (font (size 1.27 1.27)) hide)
+    )
+    (property "LCSC" "C2687423" (id 6) (at 193.675 146.05 0)
+      (effects (font (size 1.27 1.27)) hide)
+    )
+    (property "Price" "1.3917 " (id 7) (at 193.675 146.05 0)
+      (effects (font (size 1.27 1.27)) hide)
+    )
+    (pin "1")
+    (pin "2")
+    (pin "3")
+    (pin "4")
+    (pin "5")
+    (pin "6")
+    (pin "7")
+    (pin "8")
+    (pin "9")
+  )
+  (symbol (lib_id "Connector:Conn_01x02_Male") (at 231.775 146.05 180) (unit 1)
+    (in_bom yes) (on_board yes) (fields_autoplaced)
+    (property "Reference" "J?" (id 0) (at 233.045 143.5099 0)
+      (effects (font (size 1.27 1.27)) (justify right))
+    )
+    (property "Value" "Conn_01x02_Male" (id 1) (at 233.045 146.0499 0)
+      (effects (font (size 1.27 1.27)) (justify right))
+    )
+    (property "Footprint" "Connector_PinHeader_2.54mm:PinHeader_1x02_P2.54mm_Vertical" (id 2) (at 231.775 146.05 0)
+      (effects (font (size 1.27 1.27)) hide)
+    )
+    (property "Datasheet" "https://datasheet.lcsc.com/lcsc/2003141409_XFCN-PZ254V-11-02P_C492401.pdf" (id 3) (at 231.775 146.05 0)
+      (effects (font (size 1.27 1.27)) hide)
+    )
+    (property "Extended" "1" (id 4) (at 231.775 146.05 0)
+      (effects (font (size 1.27 1.27)) hide)
+    )
+    (property "LCSC" "C492401" (id 5) (at 231.775 146.05 0)
+      (effects (font (size 1.27 1.27)) hide)
+    )
+    (property "Price" "0.0149" (id 6) (at 231.775 146.05 0)
+      (effects (font (size 1.27 1.27)) hide)
+    )
+    (pin "1")
+    (pin "2")
+  )
+  (symbol (lib_id "Device:R") (at 208.915 135.255 0) (unit 1)
+    (in_bom yes) (on_board yes) (fields_autoplaced)
+    (property "Reference" "R?" (id 0) (at 211.455 133.9849 0)
+      (effects (font (size 1.27 1.27)) (justify left))
+    )
+    (property "Value" "10k" (id 1) (at 211.455 136.5249 0)
+      (effects (font (size 1.27 1.27)) (justify left))
+    )
+    (property "Footprint" "Resistor_SMD:R_0402_1005Metric" (id 2) (at 207.137 135.255 90)
+      (effects (font (size 1.27 1.27)) hide)
+    )
+    (property "Datasheet" "https://datasheet.lcsc.com/lcsc/2206010100_UNI-ROYAL-Uniroyal-Elec-0402WGF1002TCE_C25744.pdf" (id 3) (at 208.915 135.255 0)
+      (effects (font (size 1.27 1.27)) hide)
+    )
+    (property "LCSC No." "C25744" (id 4) (at 208.915 135.255 0)
+      (effects (font (size 1.27 1.27)) hide)
+    )
+    (property "Price" "0.0006" (id 5) (at 208.915 135.255 0)
+      (effects (font (size 1.27 1.27)) hide)
+    )
+    (property "Extended" "0" (id 6) (at 208.915 135.255 0)
+      (effects (font (size 1.27 1.27)) hide)
+    )
+    (property "LCSC" "C25744" (id 7) (at 208.915 135.255 0)
+      (effects (font (size 1.27 1.27)) hide)
+    )
+    (pin "1")
+    (pin "2")
+  )
+  (symbol (lib_id "Device:R") (at 217.805 135.255 0) (unit 1)
+    (in_bom yes) (on_board yes) (fields_autoplaced)
+    (property "Reference" "R?" (id 0) (at 220.345 133.9849 0)
+      (effects (font (size 1.27 1.27)) (justify left))
+    )
+    (property "Value" "10k" (id 1) (at 220.345 136.5249 0)
+      (effects (font (size 1.27 1.27)) (justify left))
+    )
+    (property "Footprint" "Resistor_SMD:R_0402_1005Metric" (id 2) (at 216.027 135.255 90)
+      (effects (font (size 1.27 1.27)) hide)
+    )
+    (property "Datasheet" "https://datasheet.lcsc.com/lcsc/2206010100_UNI-ROYAL-Uniroyal-Elec-0402WGF1002TCE_C25744.pdf" (id 3) (at 217.805 135.255 0)
+      (effects (font (size 1.27 1.27)) hide)
+    )
+    (property "LCSC No." "C25744" (id 4) (at 217.805 135.255 0)
+      (effects (font (size 1.27 1.27)) hide)
+    )
+    (property "Price" "0.0006" (id 5) (at 217.805 135.255 0)
+      (effects (font (size 1.27 1.27)) hide)
+    )
+    (property "Extended" "0" (id 6) (at 217.805 135.255 0)
+      (effects (font (size 1.27 1.27)) hide)
+    )
+    (property "LCSC" "C25744" (id 7) (at 217.805 135.255 0)
+      (effects (font (size 1.27 1.27)) hide)
+    )
+    (pin "1")
+    (pin "2")
+  )
+  (symbol (lib_id "power:GND") (at 180.34 153.67 0) (unit 1)
+    (in_bom yes) (on_board yes) (fields_autoplaced)
+    (property "Reference" "#PWR?" (id 0) (at 180.34 160.02 0)
+      (effects (font (size 1.27 1.27)) hide)
+    )
+    (property "Value" "GND" (id 1) (at 180.34 158.115 0))
+    (property "Footprint" "" (id 2) (at 180.34 153.67 0)
+      (effects (font (size 1.27 1.27)) hide)
+    )
+    (property "Datasheet" "" (id 3) (at 180.34 153.67 0)
+      (effects (font (size 1.27 1.27)) hide)
+    )
+    (pin "1")
+  )
 )

Commit message: $1
Parts:
- gave numbers to parts that had none: 4
Changed lines of the file:
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@@
   (symbol (lib_id "power:GND") (at 193.675 153.67 0) (unit 1)
     (in_bom yes) (on_board yes) (fields_autoplaced)
-    (property "Reference" "#PWR?" (id 0) (at 193.675 160.02 0)
+    (property "Reference" "#PWR0112" (id 0) (at 193.675 160.02 0)
       (effects (font (size 1.27 1.27)) hide)
     )
@@
   (symbol (lib_id "Sensor_Humidity:SHT30-DIS") (at 193.675 146.05 0) (unit 1)
     (in_bom yes) (on_board yes) (fields_autoplaced)
-    (property "Reference" "U?" (id 0) (at 195.6944 135.89 0)
+    (property "Reference" "U4" (id 0) (at 195.6944 135.89 0)
       (effects (font (size 1.27 1.27)) (justify left))
     )
@@
   (symbol (lib_id "Connector:Conn_01x02_Male") (at 231.775 146.05 180) (unit 1)
     (in_bom yes) (on_board yes) (fields_autoplaced)
-    (property "Reference" "J?" (id 0) (at 233.045 143.5099 0)
+    (property "Reference" "J3" (id 0) (at 233.045 143.5099 0)
       (effects (font (size 1.27 1.27)) (justify right))
     )
@@
   (symbol (lib_id "Device:R") (at 208.915 135.255 0) (unit 1)
     (in_bom yes) (on_board yes) (fields_autoplaced)
-    (property "Reference" "R?" (id 0) (at 211.455 133.9849 0)
+    (property "Reference" "R4" (id 0) (at 211.455 133.9849 0)
       (effects (font (size 1.27 1.27)) (justify left))
     )
@@
   (symbol (lib_id "Device:R") (at 217.805 135.255 0) (unit 1)
     (in_bom yes) (on_board yes) (fields_autoplaced)
-    (property "Reference" "R?" (id 0) (at 220.345 133.9849 0)
+    (property "Reference" "R5" (id 0) (at 220.345 133.9849 0)
       (effects (font (size 1.27 1.27)) (justify left))
     )
@@
   (symbol (lib_id "power:GND") (at 180.34 153.67 0) (unit 1)
     (in_bom yes) (on_board yes) (fields_autoplaced)
-    (property "Reference" "#PWR?" (id 0) (at 180.34 160.02 0)
+    (property "Reference" "#PWR0111" (id 0) (at 180.34 160.02 0)
       (effects (font (size 1.27 1.27)) hide)
     )

Commit message: power
Parts:
- R4, R5: LCSC No. C25744 -> (none)
Changed lines of the file:
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@@
       (effects (font (size 1.27 1.27)) hide)
     )
-    (property "LCSC No." "C25744" (id 4) (at 208.915 135.255 0)
+    (property "LCSC No." "" (id 4) (at 208.915 135.255 0)
       (effects (font (size 1.27 1.27)) hide)
     )
@@
       (effects (font (size 1.27 1.27)) hide)
     )
-    (property "LCSC No." "C25744" (id 4) (at 217.805 135.255 0)
+    (property "LCSC No." "" (id 4) (at 217.805 135.255 0)
       (effects (font (size 1.27 1.27)) hide)
     )
