File: 1. Power Submodule/Group22_Power/Sensors.kicad_sch (KiCad schematic)
At the start: 4 parts, among them J2 Conn_01x02_Male, U5 SHT30-DIS

Commit message: $1
Parts:
- U5: symbol Sensor_Humidity:SHT30-DIS -> SarahLib:SHT30-DIS
Changed lines of the file:
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@@
     (effects (font (size 1.27 1.27)) (justify left bottom))
   )
-  (global_label "+3V3Reg" (shape input) (at 208.915 125.73 180) (fields_autoplaced)
+  (hierarchical_label "+3V3Reg" (shape input) (at 208.915 125.73 180)
     (effects (font (size 1.27 1.27)) (justify right))
-    (property "Intersheet References" "${INTERSHEET_REFS}" (id 0) (at 197.9143 125.6506 0)
-      (effects (font (size 1.27 1.27)) (justify right) hide)
-    )
   )
   (symbol (lib_id "power:GND") (at 217.17 153.67 0) (unit 1)
@@
     (pin "1")
   )
-  (symbol (lib_id "Sensor_Humidity:SHT30-DIS") (at 217.17 146.05 0) (unit 1)
+  (symbol (lib_id "SarahLib:SHT30-DIS") (at 217.17 146.05 0) (unit 1)
     (in_bom yes) (on_board yes) (fields_autoplaced)
     (property "Reference" "U5" (id 0) (at 219.1894 135.89 0)

Commit message: $1
Parts:
- added J10, J11, J12, J13, J14, J15, J16, J9: Conn_01x02_Male, Connector_PinHeader_2.54mm:PinHeader_1x02_P2.54mm_Vertical, symbol Connector:Conn_01x02_Male
- J2: Extended 1 -> (none); LCSC C492401 -> (none); Price 0.0149 -> (none)
Connections:
- net +3V3Reg: now also J13.2 (Pin_2), J14.2 (Pin_2), J15.2 (Pin_2), J16.2 (Pin_2)
- net GND: now also J10.1 (Pin_1), J11.1 (Pin_1), J12.1 (Pin_1), J13.1 (Pin_1), J14.1 (Pin_1), J15.1 (Pin_1), J16.1 (Pin_1), J9.1 (Pin_1)
- new net +5VReg: J10.2 (Pin_2), J11.2 (Pin_2), J12.2 (Pin_2), J9.2 (Pin_2)
Other:
- note added: "+3V3 headers for additional sensors"
- note added: "+5V headers for scale circuit"
- moved on the sheet: J2, R8, R9, U5

Commit message: $1
Parts:
- removed J2: Conn_01x02_Male, Connector_PinHeader_2.54mm:PinHeader_1x02_P2.54mm_Vertical, symbol Connector:Conn_01x02_Male
- added J1: Conn_01x02_Male, Connector_PinHeader_2.54mm:PinHeader_1x02_P2.54mm_Vertical, symbol Connector:Conn_01x02_Male
- J10, J11, J12, J13, J14, J15, J16, J9: Populate (none) -> No
- R8, R9, U5: Populate (none) -> Yes
Connections:
- net SCL: now also J1.1 (Pin_1)
- net SDA: now also J1.2 (Pin_2)
Changed lines of the file:
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@@
+      (effects (font (size 1.27 1.27)) hide)
+    )
+    (property "Populate" "Yes" (id 8) (at 224.155 146.05 0)
       (effects (font (size 1.27 1.27)) hide)
     )
@@
       (effects (font (size 1.27 1.27)) hide)
     )
+    (property "Populate" "No" (id 7) (at 98.425 130.175 0)
+      (effects (font (size 1.27 1.27)) hide)
+    )
     (pin "1")
     (pin "2")
@@
     (pin "1")
   )
-  (symbol (lib_id "Connector:Conn_01x02_Male") (at 262.255 146.05 180) (unit 1)
-    (in_bom yes) (on_board yes) (fields_autoplaced)
-    (property "Reference" "J2" (id 0) (at 263.525 143.5099 0)
-      (effects (font (size 1.27 1.27)) (justify right))
-    )
-    (property "Value" "Conn_01x02_Male" (id 1) (at 263.525 146.0499 0)
-      (effects (font (size 1.27 1.27)) (justify right))
-    )
-    (property "Footprint" "Connector_PinHeader_2.54mm:PinHeader_1x02_P2.54mm_Vertical" (id 2) (at 262.255 146.05 0)
-      (effects (font (size 1.27 1.27)) hide)
-    )
-    (property "Datasheet" "" (id 3) (at 262.255 146.05 0)
-      (effects (font (size 1.27 1.27)) hide)
-    )
-    (property "Extended" "" (id 4) (at 262.255 146.05 0)
-      (effects (font (size 1.27 1.27)) hide)
-    )
-    (property "LCSC" "" (id 5) (at 262.255 146.05 0)
-      (effects (font (size 1.27 1.27)) hide)
-    )
-    (property "Price" "" (id 6) (at 262.255 146.05 0)
-      (effects (font (size 1.27 1.27)) hide)
-    )
-    (pin "1")
-    (pin "2")
-  )
   (symbol (lib_id "Device:R") (at 239.395 135.255 0) (unit 1)
     (in_bom yes) (on_board yes) (fields_autoplaced)
@@
       (effects (font (size 1.27 1.27)) hide)
     )
+    (property "Populate" "Yes" (id 8) (at 239.395 135.255 0)
+      (effects (font (size 1.27 1.27)) hide)
+    )
     (pin "1")
     (pin "2")
@@
       (effects (font (size 1.27 1.27)) hide)
     )
+    (property "Populate" "No" (id 7) (at 98.425 153.67 0)
+      (effects (font (size 1.27 1.27)) hide)
+    )
     (pin "1")
     (pin "2")
@@
       (effects (font (size 1.27 1.27)) hide)
     )
+    (property "Populate" "No" (id 7) (at 158.115 130.175 0)
+      (effects (font (size 1.27 1.27)) hide)
+    )
     (pin "1")
     (pin "2")
@@
       (effects (font (size 1.27 1.27)) hide)
     )
+    (property "Populate" "No" (id 7) (at 158.115 138.43 0)
+      (effects (font (size 1.27 1.27)) hide)
+    )
     (pin "1")
     (pin "2")
@@
     )
     (property "Price" "" (id 6) (at 98.425 146.05 0)
+      (effects (font (size 1.27 1.27)) hide)
+    )
+    (property "Populate" "No" (id 7) (at 98.425 146.05 0)
       (effects (font (size 1.27 1.27)) hide)
     )
@@
       (effects (font (size 1.27 1.27)) hide)
     )
+    (property "Populate" "No" (id 7) (at 98.425 138.43 0)
+      (effects (font (size 1.27 1.27)) hide)
+    )
     (pin "1")
     (pin "2")
@@
     )
     (property "Price" "" (id 6) (at 158.115 153.67 0)
+      (effects (font (size 1.27 1.27)) hide)
+    )
+    (property "Populate" "No" (id 7) (at 158.115 153.67 0)
       (effects (font (size 1.27 1.27)) hide)
     )
@@
       (effects (font (size 1.27 1.27)) hide)
     )
+    (property "Populate" "Yes" (id 8) (at 248.285 135.255 0)
+      (effects (font (size 1.27 1.27)) hide)
+    )
     (pin "1")
     (pin "2")
@@
       (effects (font (size 1.27 1.27)) hide)
     )
-    (property "LCSC" "" (id 5) (at 158.115 146.05 0)
-      (effects (font (size 1.27 1.27)) hide)
-    )
     (property "Price" "" (id 6) (at 158.115 146.05 0)
       (effects (font (size 1.27 1.27)) hide)
     )
+    (property "Populate" "No" (id 7) (at 158.115 146.05 0)
+      (effects (font (size 1.27 1.27)) hide)
+    )
+    (pin "1")
+    (pin "2")
+  )
+  (symbol (lib_id "Connector:Conn_01x02_Male") (at 262.255 146.05 180) (unit 1)
+    (in_bom yes) (on_board yes) (fields_autoplaced)
+    (property "Reference" "J1" (id 0) (at 263.525 143.5099 0)
+      (effects (font (size 1.27 1.27)) (justify right))
+    )
+    (property "Value" "Conn_01x02_Male" (id 1) (at 263.525 146.0499 0)
+      (effects (font (size 1.27 1.27)) (justify right))
+    )
+    (property "Footprint" "Connector_PinHeader_2.54mm:PinHeader_1x02_P2.54mm_Vertical" (id 2) (at 262.255 146.05 0)
+      (effects (font (size 1.27 1.27)) hide)
+    )
+    (property "Datasheet" "" (id 3) (at 262.255 146.05 0)
+      (effects (font (size 1.27 1.27)) hide)
+    )
+    (property "Extended" "" (id 4) (at 262.255 146.05 0)
+      (effects (font (size 1.27 1.27)) hide)
+    )
+    (property "Price" "" (id 6) (at 262.255 146.05 0)
+      (effects (font (size 1.27 1.27)) hide)
+    )
+    (property "Populate" "No" (id 7) (at 262.255 146.05 0)
+      (effects (font (size 1.27 1.27)) hide)
+    )
