File: 1. Power Submodule/Group22_Power/VoltageSupply.kicad_sch (KiCad schematic)
At the start: 4 parts

Commit message: $1
Parts:
- added C? (x3): 100n, Capacitor_SMD:C_0603_1608Metric, symbol Device:C_Small
- added J?: Conn_01x02_Male, symbol Connector:Conn_01x02_Male
- added U?: L78M, Package_TO_SOT_SMD:TO-252-2, symbol PCB_Library_From_Template(Stefan):HT75
- U?: value HT75 -> XC6206; footprint Project_Library:HT75 -> Package_TO_SOT_SMD:SOT-23; Alt_LCSC (none) -> C5148692; LCSC C14289 -> C347376; Price 0.2291 -> 0.0171
Connections:
- net +3V3REG: now also U?.2 (Vout), C?.1; no longer U?.3 (Vout)
- net Bat (Protected): now also U?.3 (Vin), C?.1, U?.1 (Vin); no longer U?.2 (Vin)
- net GND: now also C?.2, C?.2, C?.2, U?.2 (GND)
- new net +5VREG: C?.1, U?.3 (Vout)
Other:
- note added: "3.3V Regulation with UVLO"
- note added: "5V Regulation with UVLO"
- note removed: "Voltage Step-Down and Regulation with UVLO"
- moved on the sheet: BT?, D?, J?, U?

Commit message: power pcb
Parts:
- added BT?: Li-Ion Battery, Battery:BatteryHolder_Keystone_1042_1x18650, symbol Device:Battery_Cell
- added C?: 4.7u, Capacitor_SMD:C_1206_3216Metric, symbol Device:C_Small
- added Q?: 2N7002, Package_TO_SOT_SMD:SOT-23, symbol Transistor_FET:2N7002
- added Q?: NCE30P30K, Package_TO_SOT_SMD:TO-252-2, symbol SarahLibrary:NCE30P30K
- added R?: 82k, Resistor_SMD:R_0805_2012Metric, symbol Device:R
- added R?: 100k, Resistor_SMD:R_0402_1005Metric, symbol Device:R
- added R?: 330k, Resistor_SMD:R_0402_1005Metric, symbol Device:R
- added U?: LN61C, Package_TO_SOT_SMD:SOT-23, symbol Power_Management:BD48LxxG
- C? (x3): LCSC C14663 -> C49678
- J?: footprint (none) -> Connector_PinHeader_2.54mm:PinHeader_1x02_P2.54mm_Vertical; Extended (none) -> 1; LCSC (none) -> C492401; Price (none) -> 0.0149
- J?: Extended (none) -> 1; Price 0.0111 -> 0.0149
- U? (x2): Extended (none) -> 1
Connections:
- net +5VREG: now also J?.2 (Pin_2), Q?.3 (S), R?.1, U?.3 (VIN)
- net Bat (Protected): no longer U?.3 (Vin)
- net GND: now also BT?.2 (-), C?.2, Q?.2 (S), R?.2, U?.2 (GND); no longer BT?.2 (-)
- net at J?.1 (Pin_1): now also Q?.1 (G), R?.1, U?.1 (VOUT)
- net BAT+ renamed Bat+
- new net: Q?.1 (G), R?.1, R?.2
- new net: Q?.3 (D), R?.2
- new net: BT?.1 (+), BT?.2 (-)
- new net +5VREG(Protected): C?.1, Q?.2 (D), U?.3 (Vin)
Other:
- note added: "3.3V Regulation"
- note added: "5V Regulation"
- note added: "Undervoltage Protection"
- note removed: "3.3V Regulation with UVLO"
- note removed: "5V Regulation with UVLO"
- moved on the sheet: BT?, C?, J?, U?

Commit message: $1
Parts:
- gave numbers to parts that had none: 17
Connections:
- net Bat+: now also BT2.1 (+)
- net GND: now also BT1.2 (-)
Other:
- moved on the sheet: BT1, BT2

Commit message: power
Parts:
- added U?: TPS63030DSKR, Package_SON:WSON-10-1EP_2.5x2.5mm_P0.5mm_EP1.2x2mm, symbol SarahLib:TPS61093DSKR
- J1: Sensor_Module 1 -> (none)
Other:
- note added: "5V Boost Regulator"
- moved on the sheet: C1, C4, J2, Q1, Q2, R1, R2, R3, U1, U3

Commit message: power
Parts:
- removed C1: 100n, Capacitor_SMD:C_0603_1608Metric, symbol Device:C_Small
- removed U1: L78M, Package_TO_SOT_SMD:TO-252-2, symbol PCB_Library_From_Template(Stefan):HT75
- added C? (x4): 100n, Capacitor_SMD:C_0603_1608Metric, symbol Device:C_Small
- added C?: 1u, Capacitor_SMD:C_0805_2012Metric, symbol Device:C_Small
- added C?: 4.7u, Capacitor_SMD:C_1206_3216Metric, symbol Device:C_Small
- added L?: 10u, Inductor_SMD:L_0603_1608Metric, symbol Device:L
- added R?: 200k, Resistor_SMD:R_0805_2012Metric, symbol Device:R
- added R?: 180k, symbol Device:R
- added R?: 20k, symbol Device:R
- C2, C3: LCSC No. C49678 -> (none)
- C4: LCSC No. C29823 -> (none); Price 0.0091 -> 0.0339
- Q1: LCSC No. C8545 -> (none)
- Q2: LCSC No. C130106 -> (none)
- R1: LCSC No. C25778 -> (none)
- R2: LCSC No. C25741 -> (none)
- R3: LCSC No. C17840 -> (none)
Connections:
- net +5VREG: now also C?.2
- net Bat (Protected): now also U?.2 (VIN), U?.5 (EN), C?.1, L?.1
- net GND: now also U?.1 (GND), C?.1, C?.2
- net at U?.10 (VOUT): now also C?.1
- net at U?.3 (CP2): now also C?.2
- net at U?.4 (CP1): now also C?.1
- net at U?.6 (SS): now also C?.2
- net at U?.9 (SW): now also L?.2
Other:
- note removed: "5V Regulation"
- moved on the sheet: U?
