File: 1. Power Submodule/Group22_Power/VoltageSupply.kicad_sch (KiCad schematic)
At the start: 32 parts, among them J1 Conn_01x02_Male, U1 TPS63030DSKR, U2 HT75xx-1-SOT89, U3 USB_Micro_B_Female_Connector, U4 TP4056_1

Commit message: $1
Parts:
- removed D1: Diode, Diode_SMD:D_SOD-123, symbol Diode:1N5819
- added D4: Diode, Diode_SMD:D_SOD-123, symbol Diode:1N5819
- added J6: Conn_01x02_Male, Connector_PinHeader_2.54mm:PinHeader_1x02_P2.54mm_Vertical, symbol Connector:Conn_01x02_Male
- added J8: USB_C_Receptacle, SarahFootprints:USB-TYPE-C-TH_USB-306A-B-SU, symbol Connector:USB_C_Receptacle
- added Q1: Si2301CDS, Package_TO_SOT_SMD:SOT-23, symbol Transistor_FET:Si2319CDS
- added R10, R11: 5.1k, Resistor_SMD:R_0805_2012Metric, symbol Device:R
- added R12: 100k, Resistor_SMD:R_0402_1005Metric, symbol Device:R
- added R13: 1k, Resistor_SMD:R_0603_1608Metric, symbol Device:R
- added TP6, TP7: TestPoint, TestPoint:TestPoint_Pad_D2.0mm, symbol Connector:TestPoint
- renumbered U3 to J3
Connections:
- net +3V3Reg: now also TP5.1; no longer TP4.1
- net +5VReg: now also TP4.1; no longer TP3.1
- net Bat+: now also TP2.1, J6.1 (Pin_1), Q1.3 (D); no longer TP1.1
- net GND: now also J8.A1 (GND), J8.A12 (GND), J8.B1 (GND), J8.B12 (GND), J8.S1 (SHIELD), R10.1, R11.1, R12.1, TP6.1; no longer TP5.1
- net VUSB: now also TP1.1, D4.2 (A), J8.A4 (VBUS), J8.A9 (VBUS), J8.B4 (VBUS), J8.B9 (VBUS), Q1.1 (G), R12.2
- net at J1.2 (Pin_2): now also D4.1 (K), J6.2 (Pin_2), Q1.2 (S)
- net Bat(Protected) renamed Power
- net Power: now also TP3.1, R13.2; no longer TP2.1, U1.5 (EN)
- new net: R13.1, TP7.1, U1.5 (EN)
- new net: J8.B5 (CC2), R10.2
- new net: J8.A5 (CC1), R11.2
- no-connect marks 2 -> 16
Other:
- note added: "Input Polarity Protection and charging switching"
- note added: "Micro-USB Connector"
- note added: "USB C Connector"
- note removed: "Input Polarity Protection"
- note removed: "USB Connector"
- moved on the sheet: C6, C7, C8, C9, D2, D3, J1, J3, R4, R5, R6, R7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

Commit message: $1
Parts:
- J1, J6: Extended 1 -> (none); LCSC C492401 -> (none); Price 0.0149 -> (none)
Connections:
- net Reg: now reaches R13.1, TP7.1, U1.5 (EN)
Changed lines of the file:
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@@
     (effects (font (size 2 2) (thickness 0.8) bold) (justify left bottom))
+  )
+  (label "Reg" (at 24.13 93.345 0)
+    (effects (font (size 1.27 1.27)) (justify left bottom))
   )
   (label "Power" (at 19.685 69.215 180)
@@
       (effects (font (size 1.27 1.27)) hide)
     )
-    (property "Datasheet" "https://datasheet.lcsc.com/lcsc/2003141409_XFCN-PZ254V-11-02P_C492401.pdf" (id 3) (at 106.68 31.115 0)
-      (effects (font (size 1.27 1.27)) hide)
-    )
-    (property "LCSC" "C492401" (id 4) (at 106.68 31.115 0)
-      (effects (font (size 1.27 1.27)) hide)
-    )
-    (property "Price" "0.0149" (id 5) (at 106.68 31.115 0)
+    (property "Datasheet" "" (id 3) (at 106.68 31.115 0)
+      (effects (font (size 1.27 1.27)) hide)
+    )
+    (property "LCSC" "" (id 4) (at 106.68 31.115 0)
+      (effects (font (size 1.27 1.27)) hide)
+    )
+    (property "Price" "" (id 5) (at 106.68 31.115 0)
       (effects (font (size 1.27 1.27)) hide)
     )
@@
       (effects (font (size 1.27 1.27)) hide)
     )
-    (property "Extended" "1" (id 7) (at 106.68 31.115 0)
+    (property "Extended" "" (id 7) (at 106.68 31.115 0)
       (effects (font (size 1.27 1.27)) hide)
     )
@@
       (effects (font (size 1.27 1.27)) hide)
     )
-    (property "Datasheet" "https://datasheet.lcsc.com/lcsc/2003141409_XFCN-PZ254V-11-02P_C492401.pdf" (id 3) (at 96.52 50.165 0)
-      (effects (font (size 1.27 1.27)) hide)
-    )
-    (property "LCSC" "C492401" (id 4) (at 96.52 50.165 0)
-      (effects (font (size 1.27 1.27)) hide)
-    )
-    (property "Price" "0.0149" (id 5) (at 96.52 50.165 0)
+    (property "Datasheet" "" (id 3) (at 96.52 50.165 0)
+      (effects (font (size 1.27 1.27)) hide)
+    )
+    (property "LCSC" "" (id 4) (at 96.52 50.165 0)
+      (effects (font (size 1.27 1.27)) hide)
+    )
+    (property "Price" "" (id 5) (at 96.52 50.165 0)
       (effects (font (size 1.27 1.27)) hide)
     )
@@
       (effects (font (size 1.27 1.27)) hide)
     )
-    (property "Extended" "1" (id 7) (at 96.52 50.165 0)
-      (effects (font (size 1.27 1.27)) hide)
-    )
+    (property "Extended" "" (id 7) (at 96.52 50.165 0)
+      (effects (font (size 1.27 1.27)) hide)
+    )

Commit message: $1
Parts:
- removed J1, J6: Conn_01x02_Male, Connector_PinHeader_2.54mm:PinHeader_1x02_P2.54mm_Vertical, symbol Connector:Conn_01x02_Male
- added JP1, JP2: Jumper_2_Open, Jumper:SolderJumper-2_P1.3mm_Open_RoundedPad1.0x1.5mm, symbol Jumper:Jumper_2_Open
Connections:
- net Bat+: now also JP1.1 (A)
- net Power: now also JP2.2 (B)
- net at D4.1 (K), Q1.2 (S): now also JP1.2 (B), JP2.1 (A)
Other:
- moved on the sheet: C6

Commit message: $1
Parts:
- BT1, BT2: Populate (none) -> No
- C1, C8, C9, D2, D3, J8, L1, Q1, R1, R10, R11, R13, R2, R3, R4, R5, R6, R7, U2, U4: Populate (none) -> Yes
- R12: LCSC (none) -> C25741; LCSC No. C25741 -> (none); Populate (none) -> Yes
Changed lines of the file:
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@@
+      (effects (font (size 1.27 1.27)) hide)
+    )
+    (property "Populate" "Yes" (id 8) (at 24.13 108.585 0)
       (effects (font (size 1.27 1.27)) hide)
     )
@@
     )
     (property "Extended" "0" (id 6) (at 188.595 80.01 0)
+      (effects (font (size 1.27 1.27)) hide)
+    )
+    (property "Populate" "Yes" (id 7) (at 188.595 80.01 0)
       (effects (font (size 1.27 1.27)) hide)
     )
@@
       (effects (font (size 1.27 1.27)) hide)
     )
+    (property "Populate" "Yes" (id 8) (at 120.015 71.12 0)
+      (effects (font (size 1.27 1.27)) hide)
+    )
     (pin "1")
     (pin "2")
@@
       (effects (font (size 1.27 1.27)) hide)
     )
+    (property "Populate" "No" (id 4) (at 37.465 32.385 0)
+      (effects (font (size 1.27 1.27)) hide)
+    )
     (pin "1")
     (pin "2")
@@
     )
     (property "Price" "0.01" (id 6) (at 76.835 99.06 0)
+      (effects (font (size 1.27 1.27)) hide)
+    )
+    (property "Populate" "Yes" (id 7) (at 76.835 99.06 0)
       (effects (font (size 1.27 1.27)) hide)
     )
@@
       (effects (font (size 1.27 1.27)) hide)
     )
+    (property "Populate" "Yes" (id 7) (at 145.415 76.2 0)
+      (effects (font (size 1.27 1.27)) hide)
+    )
     (pin "1")
     (pin "2")
@@
       (effects (font (size 1.27 1.27)) hide)
     )
+    (property "Populate" "Yes" (id 7) (at 53.34 69.215 0)
+      (effects (font (size 1.27 1.27)) hide)
+    )
     (pin "1")
     (pin "2")
@@
     )
     (property "LCSC" "C1779" (id 7) (at 34.925 73.025 0)
+      (effects (font (size 1.27 1.27)) hide)
+    )
+    (property "Populate" "Yes" (id 8) (at 34.925 73.025 0)
       (effects (font (size 1.27 1.27)) hide)
     )
@@
     )
     (property "LCSC" "C27834" (id 7) (at 264.16 39.37 0)
+      (effects (font (size 1.27 1.27)) hide)
+    )
+    (property "Populate" "Yes" (id 8) (at 264.16 39.37 0)
       (effects (font (size 1.27 1.27)) hide)
     )
@@
       (effects (font (size 1.27 1.27)) hide)
     )
-    (property "LCSC No." "C25741" (id 4) (at 81.915 26.035 0)
+    (property "LCSC No." "" (id 4) (at 81.915 26.035 0)
       (effects (font (size 1.27 1.27)) hide)
     )
@@
     )
     (property "Extended" "0" (id 6) (at 81.915 26.035 0)
+      (effects (font (size 1.27 1.27)) hide)
+    )
+    (property "LCSC" "C25741" (id 7) (at 81.915 26.035 0)
+      (effects (font (size 1.27 1.27)) hide)
+    )
+    (property "Populate" "Yes" (id 8) (at 81.915 26.035 0)
       (effects (font (size 1.27 1.27)) hide)
     )
@@
       (effects (font (size 1.27 1.27)) hide)
     )
+    (property "Populate" "No" (id 4) (at 15.875 32.385 0)
+      (effects (font (size 1.27 1.27)) hide)
+    )
     (pin "1")
     (pin "2")
@@
     )
     (property "Extended" "0" (id 6) (at 145.415 85.09 0)
+      (effects (font (size 1.27 1.27)) hide)
+    )
+    (property "Populate" "Yes" (id 7) (at 145.415 85.09 0)
       (effects (font (size 1.27 1.27)) hide)
     )
@@
       (effects (font (size 1.27 1.27)) hide)
     )
+    (property "Populate" "Yes" (id 6) (at 159.385 32.385 0)
+      (effects (font (size 1.27 1.27)) hide)
+    )
     (pin "1")
     (pin "2")
@@
       (effects (font (size 1.27 1.27)) hide)
     )
+    (property "Populate" "Yes" (id 7) (at 136.525 76.2 0)
+      (effects (font (size 1.27 1.27)) hide)
+    )
     (pin "1")
     (pin "2")
@@
       (effects (font (size 1.27 1.27)) hide)
     )
+    (property "Populate" "Yes" (id 8) (at 272.415 39.37 0)
+      (effects (font (size 1.27 1.27)) hide)
+    )
     (pin "1")
     (pin "2")
@@
     )
     (property "Extended" "0" (id 6) (at 24.13 78.105 0)
+      (effects (font (size 1.27 1.27)) hide)
+    )
+    (property "Populate" "Yes" (id 7) (at 24.13 78.105 0)
       (effects (font (size 1.27 1.27)) hide)
     )
@@
       (effects (font (size 1.27 1.27)) hide)
     )
+    (property "Populate" "Yes" (id 5) (at 89.535 33.655 0)
+      (effects (font (size 1.27 1.27)) hide)
+    )
     (pin "1")
     (pin "2")
@@
       (effects (font (size 1.27 1.27)) hide)
     )
+    (property "Populate" "Yes" (id 7) (at 127.635 85.09 0)
+      (effects (font (size 1.27 1.27)) hide)
+    )
     (pin "1")
     (pin "2")
@@
       (effects (font (size 1.27 1.27)) hide)
     )
+    (property "Populate" "Yes" (id 7) (at 76.835 109.855 0)
+      (effects (font (size 1.27 1.27)) hide)
+    )
     (pin "1")
     (pin "2")
@@
     )
     (property "Extended" "0" (id 6) (at 136.525 85.09 0)
+      (effects (font (size 1.27 1.27)) hide)
+    )
+    (property "Populate" "Yes" (id 7) (at 136.525 85.09 0)
       (effects (font (size 1.27 1.27)) hide)
     )
@@
     )
     (property "LCSC" "C309339" (id 4) (at 243.84 53.34 0)
+      (effects (font (size 1.27 1.27)) hide)
+    )
+    (property "Populate" "Yes" (id 5) (at 243.84 53.34 0)
       (effects (font (size 1.27 1.27)) hide)
     )
@@
       (effects (font (size 1.27 1.27)) hide)
     )
+    (property "Populate" "Yes" (id 7) (at 167.005 73.66 0)
+      (effects (font (size 1.27 1.27)) hide)
+    )
     (pin "1")
     (pin "2")
@@
       (effects (font (size 1.27 1.27)) hide)
     )
+    (property "Populate" "Yes" (id 8) (at 180.34 100.33 0)
+      (effects (font (size 1.27 1.27)) hide)
+    )

Commit message: $1
Parts:
- U1: value TPS63030DSKR -> TPS61093
Changed lines of the file:
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@@
     (in_bom yes) (on_board yes) (fields_autoplaced)
     (property "Reference" "U1" (id 0) (at 53.34 78.74 0))
-    (property "Value" "TPS63030DSKR" (id 1) (at 53.34 81.28 0))
+    (property "Value" "TPS61093" (id 1) (at 53.34 81.28 0))
     (property "Footprint" "Package_SON:WSON-10-1EP_2.5x2.5mm_P0.5mm_EP1.2x2mm" (id 2) (at 87.63 114.3 0)
       (effects (font (size 1.27 1.27)) hide)
     )
-    (property "Datasheet" "http://www.ti.com/lit/ds/symlink/tps63030.pdf" (id 3) (at 64.77 63.5 0)
+    (property "Datasheet" "https://datasheet.lcsc.com/lcsc/1806081810_Texas-Instruments-TPS61093DSKR_C60707.pdf" (id 3) (at 64.77 63.5 0)
       (effects (font (size 1.27 1.27)) hide)
     )

Commit message: power:
Other:
- moved on the sheet: BT1, BT2, C1, C2, C3, C4, C5, C6, C7, C8, C9, D2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

Commit message: $1
Other:
- moved on the sheet: C1, C2, C3, C4, C5, C7, L1, R1, R13, R2, R3, TP7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
