File: 1. Power Submodule/Group22_Power/Group22_Power.kicad_pcb (KiCad board)
At the start: 2 copper layers, 100 x 79.2 mm, 36 parts, among them J1 Conn_01x02_Male, J2 Conn_01x02_Male, U1 TPS63030DSKR, U2 HT75xx-1-SOT89, U3 USB_Micro_B_Female_Connector, U4 TP4056_1, U5 SHT30-DIS

Commit message: $1
Parts:
- removed D1: Diode, Diode_SMD:D_SOD-123
- removed U3: USB_Micro_B_Female_Connector, SarahFootprints:C404969_Micro_USB
- added D4: Diode, Diode_SMD:D_SOD-123, F.Cu at (103.4, 98.5)
- added J3: USB_Micro_B_Female_Connector, SarahFootprints:C404969_Micro_USB, F.Cu at (57.6, 105.9)
- added J4: Conn_01x08_Male, Connector_PinHeader_2.54mm:PinHeader_1x08_P2.54mm_Vertical, F.Cu at (196.0, 46.6)
- added J5: Conn_01x08_Male, Connector_PinHeader_2.54mm:PinHeader_1x08_P2.54mm_Vertical, F.Cu at (191.4, 46.6)
- added J6: Conn_01x02_Male, Connector_PinHeader_2.54mm:PinHeader_1x02_P2.54mm_Vertical, F.Cu at (100.2, 103.8)
- added J7: GPIO, Connector_PinSocket_2.54mm:PinSocket_2x20_P2.54mm_Vertical, F.Cu at (186.8, 46.6)
- added J8: USB_C_Receptacle, SarahFootprints:USB-TYPE-C-TH_USB-306A-B-SU, F.Cu at (63.1, 120.7)
- added Q1: Si2301CDS, Package_TO_SOT_SMD:SOT-23, F.Cu at (97.8, 97.8)
- added R10: 5.1k, Resistor_SMD:R_0805_2012Metric, F.Cu at (69.7, 123.0)
- added R11: 5.1k, Resistor_SMD:R_0805_2012Metric, F.Cu at (69.7, 120.0)
- added R12: 100k, Resistor_SMD:R_0402_1005Metric, F.Cu at (101.7, 99.2)
- added R13: 1k, Resistor_SMD:R_0603_1608Metric, F.Cu at (116.8, 106.5)
- added TP6: TestPoint, TestPoint:TestPoint_Pad_D2.0mm, F.Cu at (115.2, 116.5)
- added TP7: TestPoint, TestPoint:TestPoint_Pad_D2.0mm, F.Cu at (119.8, 114.8)
- moved C6 21.9 mm to (110.6, 99.7), turned to 0 degrees
- moved J1 20.4 mm to (109.8, 96.8)
- moved C1 18.1 mm to (116.7, 99.9)
- moved C2 18.1 mm to (121.2, 106.0)
- moved C5 18.1 mm to (125.9, 103.9)
- moved L1 18.1 mm to (120.7, 97.0)
- moved R1 18.1 mm to (119.3, 106.2)
- moved R2 18.1 mm to (124.0, 103.7)
- moved R3 18.1 mm to (124.8, 106.6)
- moved U1 18.1 mm to (120.0, 102.9)
- moved C3 18.1 mm to (116.8, 104.2)
- moved C4 18.1 mm to (120.4, 100.5)
- moved C7 18.1 mm to (136.4, 96.7)
- moved J2 18.1 mm to (144.4, 103.9)
- moved R8 18.1 mm to (144.6, 99.9)
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Connections:
- BT1 pad 1: Bat+ -> /VoltageSupply/Bat+
- BT2 pad 1: Bat+ -> /VoltageSupply/Bat+
- C1 pad 1: Bat(Protected) -> /VoltageSupply/Power
- C5 pad 2: +5VReg -> /Microcontrollers/+5VReg
- C6 pad 1: Bat(Protected) -> /VoltageSupply/Power
- C7 pad 1: +3V3Reg -> /Sensors/+3V3Reg
- C9 pad 1: Bat+ -> /VoltageSupply/Bat+
- J1 pad 1: Bat(Protected) -> /VoltageSupply/Power
- L1 pad 1: Bat(Protected) -> /VoltageSupply/Power
- R2 pad 1: +5VReg -> /Microcontrollers/+5VReg
- R8 pad 1: +3V3Reg -> /Sensors/+3V3Reg
- R9 pad 1: +3V3Reg -> /Sensors/+3V3Reg
- TP1 pad 1: Bat+ -> /VoltageSupply/VUSB
- TP2 pad 1: Bat(Protected) -> /VoltageSupply/Bat+
- TP3 pad 1: +5VReg -> /VoltageSupply/Power
- TP4 pad 1: +3V3Reg -> /Microcontrollers/+5VReg
- TP5 pad 1: GND -> /Sensors/+3V3Reg
- U1 pad 2: Bat(Protected) -> /VoltageSupply/Power
- U1 pad 5: Bat(Protected) -> Net-(U1-Pad5)
- U1 pad 8: +5VReg -> /Microcontrollers/+5VReg
- U2 pad 2: +5VReg -> /Microcontrollers/+5VReg
- U2 pad 3: +3V3Reg -> /Sensors/+3V3Reg
- U4 pad 5: Bat+ -> /VoltageSupply/Bat+
- U5 pad 5: +3V3Reg -> /Sensors/+3V3Reg
Routing:
- net /VoltageSupply/Bat+: track 0.00 -> 76.4 mm
- net Bat+: track 59.5 -> 0.00 mm
- net Bat(Protected): track 25.2 -> 0.00 mm
- net /VoltageSupply/Power: track 0.00 -> 21.6 mm
- net +5VReg: track 16.6 -> 0.00 mm
- net /Microcontrollers/+5VReg: track 0.00 -> 16.6 mm
- net /Sensors/+3V3Reg: track 0.00 -> 15.9 mm
- net +3V3Reg: track 15.9 -> 0.00 mm
- net Net-(J1-Pad2): track 3.18 -> 18.8 mm
- net Net-(J8-PadB5): track 0.00 -> 13.8 mm
- net Net-(C8-Pad1): track 37.2 -> 25.7 mm
- net /VoltageSupply/VUSB: track 2.90 -> 11.2 mm
- net Net-(R5-Pad2): track 3.51 -> 0.00 mm
- net Net-(U1-Pad5): track 0.00 -> 3.10 mm
- net Net-(R6-Pad2): track 2.62 -> 0.01 mm
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Other:
- board size 100 x 79.2 mm -> 100 x 88.8 mm
- board text added: "Board by Sarah Tallack Group 22 EEE4113F Power Submodule Version 1"
- board text added: "Charging (RED)"
- board text added: "Charging Done (YELLOW)"
- board text added: "Protection and switching"
- board text added: "USB Charger"
- board text removed: "Micro-USB Charger"

Commit message: $1
Parts:
- added G***: LOGO, LOGO, B.Cu at (105.5, 73.8)
- added J10: Conn_01x02_Male, Connector_PinHeader_2.54mm:PinHeader_1x02_P2.54mm_Vertical, F.Cu at (128.5, 113.6)
- added J11: Conn_01x02_Male, Connector_PinHeader_2.54mm:PinHeader_1x02_P2.54mm_Vertical, F.Cu at (128.5, 117.4)
- added J12: Conn_01x02_Male, Connector_PinHeader_2.54mm:PinHeader_1x02_P2.54mm_Vertical, F.Cu at (128.5, 121.2)
- added J13: Conn_01x02_Male, Connector_PinHeader_2.54mm:PinHeader_1x02_P2.54mm_Vertical, F.Cu at (141.0, 109.5)
- added J14: Conn_01x02_Male, Connector_PinHeader_2.54mm:PinHeader_1x02_P2.54mm_Vertical, F.Cu at (141.0, 113.3)
- added J15: Conn_01x02_Male, Connector_PinHeader_2.54mm:PinHeader_1x02_P2.54mm_Vertical, F.Cu at (141.0, 117.1)
- added J16: Conn_01x02_Male, Connector_PinHeader_2.54mm:PinHeader_1x02_P2.54mm_Vertical, F.Cu at (141.0, 120.9)
- added J9: Conn_01x02_Male, Connector_PinHeader_2.54mm:PinHeader_1x02_P2.54mm_Vertical, F.Cu at (128.5, 109.8)
- J4, J5: footprint Connector_PinHeader_2.54mm:PinHeader_1x08_P2.54mm_Vertical -> Connector_PinSocket_2.54mm:PinSocket_1x08_P2.54mm_Vertical; moved to B.Cu
- J7: moved to B.Cu
- moved J5 141.9 mm to (69.9, 119.9), turned to 180 degrees
- moved J4 126.6 mm to (92.7, 119.9), turned to 180 degrees
- moved J7 96.1 mm to (149.5, 135.2), turned to 90 degrees
- moved D2 22.7 mm to (80.2, 111.2), turned to 0 degrees
- moved D3 18.6 mm to (80.3, 106.1), turned to 0 degrees
- moved R5 17.8 mm to (76.6, 111.1), turned to 180 degrees
- moved TP7 17.0 mm to (103.0, 111.7)
- moved R6 12.7 mm to (77.1, 106.1), turned to 180 degrees
- moved R11 11.9 mm to (69.1, 108.1), turned to -90 degrees
- moved J8 11.0 mm to (63.2, 109.7)
- moved J1 10.4 mm to (99.7, 94.4)
- moved C6 10.4 mm to (100.5, 97.2)
- moved D4 10.4 mm to (93.3, 96.0)
- moved J6 10.4 mm to (90.1, 101.3)
- moved Q1 10.4 mm to (87.7, 95.3)
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Connections:
- net Net-(U1-Pad5) renamed /VoltageSupply/Reg
- J4 pad 1: /Microcontrollers/GPIO4 -> /Microcontrollers/+5VReg
- J4 pad 2: /Microcontrollers/GPIO2 -> GND
- J4 pad 3: /Microcontrollers/GPIO14 -> /Microcontrollers/GPIO12
- J4 pad 4: /Microcontrollers/GPIO15 -> /Microcontrollers/GPIO13
- J4 pad 5: /Microcontrollers/GPIO13 -> /Microcontrollers/GPIO15
- J4 pad 6: /Microcontrollers/GPIO12 -> /Microcontrollers/GPIO14
- J4 pad 7: GND -> /Microcontrollers/GPIO2
- J4 pad 8: /Microcontrollers/+5VReg -> /Microcontrollers/GPIO4
Routing:
- net /Microcontrollers/+5VReg: track 16.6 -> 137.9 mm
- net /Sensors/+3V3Reg: track 15.9 -> 79.9 mm, vias 0 -> 1
- net /VoltageSupply/VUSB: track 11.2 -> 51.1 mm, vias 0 -> 1
- net Net-(R5-Pad2): track 0.00 -> 20.2 mm, vias 0 -> 2
- net /VoltageSupply/Power: track 21.6 -> 37.5 mm
- net Net-(R6-Pad2): track 0.01 -> 13.6 mm, vias 0 -> 2
- net /VoltageSupply/Reg: track 3.10 -> 14.6 mm
- net Net-(C8-Pad1): track 25.7 -> 33.3 mm
- net /VoltageSupply/Bat+: track 76.4 -> 79.5 mm
- net Net-(J8-PadB5): track 13.8 -> 12.6 mm
- net GND: vias 2 -> 1
Other:
- board size 100 x 88.8 mm -> 100 x 100 mm
- board text added: "+3V3 supply"
- board text added: "+5V supply"
- board text added: "ESP32 CAM"
- board text added: "Power"
- board text added: "Raspberry Pi Zero W"
- board text added: "Reg"
- board text added: "VUSB"
- board text removed: "Bat(Prot)"

Commit message: $1
Parts:
- removed the G*** at (105.5, 73.8)
- removed J1, J6: Conn_01x02_Male, Connector_PinHeader_2.54mm:PinHeader_1x02_P2.54mm_Vertical
- added G***: LOGO, LOGO, F.Cu at (81.5, 129.5)
- added G***: LOGO, LOGO, F.Cu at (101.0, 124.2)
- added G***: LOGO, LOGO, B.Cu at (81.4, 128.7)
- added G***: LOGO, LOGO, B.Cu at (114.0, 85.5)
- added JP1: Jumper_2_Open, Jumper:SolderJumper-2_P1.3mm_Open_RoundedPad1.0x1.5mm, F.Cu at (90.8, 101.2)
- added JP2: Jumper_2_Open, Jumper:SolderJumper-2_P1.3mm_Open_RoundedPad1.0x1.5mm, F.Cu at (97.6, 94.4)
- moved R7 0.93 mm to (79.8, 98.3), turned to 0 degrees
Routing:
- net /VoltageSupply/VUSB: track 51.1 -> 94.9 mm, vias 1 -> 2
- net /Microcontrollers/+3V3: track 0.00 -> 21.7 mm
- net GND: track 9.66 -> 22.0 mm, vias 1 -> 2
- net /VoltageSupply/Power: track 37.5 -> 38.9 mm
- net Net-(D4-Pad1): track 18.8 -> 20.1 mm
- net Net-(C8-Pad1): track 33.3 -> 33.2 mm, vias 0 -> 2
Other:
- board text added: "Board by Sarah Tallack, Group 22, EEE4113F Power Submodule, Version 1"
- board text added: "Sarah Tallack EEE4113F Group 22"
- board text removed: "Board by Sarah Tallack Group 22 EEE4113F Power Submodule Version 1"

Commit message: pcb done
Other:
- board text added: "April 2023"
Changed lines of the file:
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@@
     (effects (font (size 0.6 0.6) (thickness 0.15)))
+  )
+  (gr_text "April 2023" (at 154.94 96.52 90) (layer "F.SilkS")
+    (effects (font (size 1 1) (thickness 0.15)))
   )
   (gr_text "3V3 Regulation" (at 126.25 106) (layer "F.SilkS")

Commit message: $1
Parts:
- removed J2: Conn_01x02_Male, Connector_PinHeader_2.54mm:PinHeader_1x02_P2.54mm_Vertical
- added J1: Conn_01x02_Male, Connector_PinHeader_2.54mm:PinHeader_1x02_P2.54mm_Vertical, F.Cu at (141.5, 99.5)
